Commit message: added robotiq gripper to ur5
Signed-off-by: Roshan Kumar <rkroshan.1999@gmail.com>

File: urdf/inc/ur_transmissions.xacro (robot description, xacro)
@@ -6,5 +6,5 @@
           this location. Nor can they rely on the existence of the macro.
   -->
-  <xacro:macro name="ur_arm_transmission" params="prefix hw_interface">
+  <xacro:macro name="ur_arm_transmission" params="prefix hw_interface EE_robotiq">
     <transmission name="${prefix}shoulder_pan_trans">
       <type>transmission_interface/SimpleTransmission</type>
@@ -61,4 +61,60 @@
       </actuator>
     </transmission>
+   <xacro:if value="${EE_robotiq}">
+      <transmission name="${prefix}robotiq_85_left_knuckle_trans">
+        <type>transmission_interface/SimpleTransmission</type>
+        <joint name="${prefix}robotiq_85_left_knuckle_joint">
+          <hardwareInterface>hardware_interface/PositionJointInterface</hardwareInterface>
+        </joint>
+        <actuator name="${prefix}robotiq_85_left_knuckle_motor">
+          <mechanicalReduction>1</mechanicalReduction>
+        </actuator>
+      </transmission>
+      <transmission name="${prefix}robotiq_85_right_knuckle_trans">
+        <type>transmission_interface/SimpleTransmission</type>
+        <joint name="${prefix}robotiq_85_right_knuckle_joint">
+          <hardwareInterface>hardware_interface/PositionJointInterface</hardwareInterface>
+        </joint>
+        <actuator name="${prefix}robotiq_85_right_knuckle_motor">
+          <mechanicalReduction>1</mechanicalReduction>
+        </actuator>
+      </transmission>
+      <transmission name="${prefix}robotiq_85_left_inner_knuckle_trans">
+        <type>transmission_interface/SimpleTransmission</type>
+        <joint name="${prefix}robotiq_85_left_inner_knuckle_joint">
+          <hardwareInterface>hardware_interface/PositionJointInterface</hardwareInterface>
+        </joint>
+        <actuator name="${prefix}robotiq_85_left_inner_knuckle_motor">
+          <mechanicalReduction>1</mechanicalReduction>
+        </actuator>
+      </transmission>
+      <transmission name="${prefix}robotiq_85_right_inner_knuckle_trans">
+        <type>transmission_interface/SimpleTransmission</type>
+        <joint name="${prefix}robotiq_85_right_inner_knuckle_joint">
+          <hardwareInterface>hardware_interface/PositionJointInterface</hardwareInterface>
+        </joint>
+        <actuator name="${prefix}robotiq_85_right_inner_knuckle_motor">
+          <mechanicalReduction>1</mechanicalReduction>
+        </actuator>
+      </transmission>
+      <transmission name="${prefix}robotiq_85_left_finger_tip_trans">
+        <type>transmission_interface/SimpleTransmission</type>
+        <joint name="${prefix}robotiq_85_left_finger_tip_joint">
+          <hardwareInterface>hardware_interface/PositionJointInterface</hardwareInterface>
+        </joint>
+        <actuator name="${prefix}robotiq_85_left_finger_tip_motor">
+          <mechanicalReduction>1</mechanicalReduction>
+        </actuator>
+      </transmission>
+      <transmission name="${prefix}robotiq_85_right_finger_tip_trans">
+        <type>transmission_interface/SimpleTransmission</type>
+        <joint name="${prefix}robotiq_85_right_finger_tip_joint">
+          <hardwareInterface>hardware_interface/PositionJointInterface</hardwareInterface>
+        </joint>
+        <actuator name="${prefix}robotiq_85_right_finger_tip_motor">
+          <mechanicalReduction>1</mechanicalReduction>
+        </actuator>
+      </transmission>
+    </xacro:if>
   </xacro:macro>
 </robot>

File: urdf/ur.ros2_control.xacro (robot description, xacro)
@@ -21,4 +21,5 @@
     non_blocking_read:=true
     keep_alive_count:=2
+    EE_robotiq
     ">
     <ros2_control name="${name}" type="system">
@@ -257,4 +258,96 @@
         </gpio>
       </xacro:unless>
+      <xacro:if value="${EE_robotiq}">
+        <joint name="${tf_prefix}robotiq_85_left_knuckle_joint">
+          <command_interface name="position">
+            <param name="min">-0.05</param>
+            <param name="max">0.80285</param>
+          </command_interface>
+          <command_interface name="velocity">
+            <param name="min">0.5</param>
+            <param name="max">0.5</param>
+          </command_interface>
+          <state_interface name="position">
+            <param name="initial_value">0.0</param>
+          </state_interface>
+          <state_interface name="velocity"/>
+          <state_interface name="effort"/>
+        </joint>
+        <joint name="${tf_prefix}robotiq_85_right_knuckle_joint">
+          <command_interface name="position">
+            <param name="min">-0.05</param>
+            <param name="max">0.80285</param>
+          </command_interface>
+          <command_interface name="velocity">
+            <param name="min">0.5</param>
+            <param name="max">0.5</param>
+          </command_interface>
+          <state_interface name="position">
+            <param name="initial_value">0.0</param>
+          </state_interface>
+          <state_interface name="velocity"/>
+          <state_interface name="effort"/>
+        </joint>
+        <joint name="${tf_prefix}robotiq_85_left_inner_knuckle_joint">
+          <command_interface name="position">
+            <param name="min">-0.05</param>
+            <param name="max">0.80285</param>
+          </command_interface>
+          <command_interface name="velocity">
+            <param name="min">0.5</param>
+            <param name="max">0.5</param>
+          </command_interface>
+          <state_interface name="position">
+            <param name="initial_value">0.0</param>
+          </state_interface>
+          <state_interface name="velocity"/>
+          <state_interface name="effort"/>
+        </joint>
+        <joint name="${tf_prefix}robotiq_85_right_inner_knuckle_joint">
+          <command_interface name="position">
+            <param name="min">-0.05</param>
+            <param name="max">0.80285</param>
+          </command_interface>
+          <command_interface name="velocity">
+            <param name="min">0.5</param>
+            <param name="max">0.5</param>
+          </command_interface>
+          <state_interface name="position">
+            <param name="initial_value">0.0</param>
+          </state_interface>
+          <state_interface name="velocity"/>
+          <state_interface name="effort"/>
+        </joint>
+        <joint name="${tf_prefix}robotiq_85_left_finger_tip_joint">
+          <command_interface name="position">
+            <param name="min">-0.80285</param>
+            <param name="max">0.05</param>
+          </command_interface>
+          <command_interface name="velocity">
+            <param name="min">0.5</param>
+            <param name="max">0.5</param>
+          </command_interface>
+          <state_interface name="position">
+            <param name="initial_value">0.0</param>
+          </state_interface>
+          <state_interface name="velocity"/>
+          <state_interface name="effort"/>
+        </joint>
+        <joint name="${tf_prefix}robotiq_85_right_finger_tip_joint">
+          <command_interface name="position">
+            <param name="min">-0.80285</param>
+            <param name="max">0.05</param>
+          </command_interface>
+          <command_interface name="velocity">
+            <param name="min">0.5</param>
+            <param name="max">0.5</param>
+          </command_interface>
+          <state_interface name="position">
+            <param name="initial_value">0.0</param>
+          </state_interface>
+          <state_interface name="velocity"/>
+          <state_interface name="effort"/>
+        </joint>
+      </xacro:if>
     </ros2_control>
   </xacro:macro>

File: urdf/ur.urdf.xacro (robot description, xacro)
@@ -9,4 +9,5 @@
    <xacro:arg name="ur_type" default="ur5x"/>
    <!-- parameters -->
+   <xacro:arg name="EE_robotiq" default="true"/>
    <xacro:arg name="tf_prefix" default="" />
    <xacro:arg name="joint_limit_params" default="$(find ur_description)/config/$(arg ur_type)/joint_limits.yaml"/>
@@ -56,4 +57,5 @@
      tf_prefix="$(arg tf_prefix)"
      parent="world"
+     EE_robotiq="$(arg EE_robotiq)"
      joint_limits_parameters_file="$(arg joint_limit_params)"
      kinematics_parameters_file="$(arg kinematics_params)"
@@ -97,5 +99,6 @@
     <gazebo>
       <plugin filename="libgazebo_ros2_control.so" name="gazebo_ros2_control">
-        <parameters>$(arg simulation_controllers)</parameters>
+        <robot_sim_type>gazebo_ros2_control/GazeboSystem</robot_sim_type>
+        <parameters>$(find ur_description)/config/urrobotiq_controller.yaml</parameters>
       </plugin>
     </gazebo>
