Commit message: added robotiq gripper to ur5
Signed-off-by: Roshan Kumar <rkroshan.1999@gmail.com>

File: urdf/ur_macro.xacro (robot description, xacro)
@@ -50,4 +50,5 @@
     *origin
     joint_limits_parameters_file
+    EE_robotiq
     kinematics_parameters_file
     physical_parameters_file
@@ -99,4 +100,5 @@
         name="${name}"
         use_fake_hardware="${use_fake_hardware}"
+        EE_robotiq="${EE_robotiq}"
         initial_positions="${initial_positions}"
         fake_sensor_commands="${fake_sensor_commands}"
@@ -129,5 +131,5 @@
     </xacro:if>
     <!-- Add URDF transmission elements (for ros_control) -->
-    <!--<xacro:ur_arm_transmission prefix="${prefix}" hw_interface="${transmission_hw_interface}" />-->
+    <!--<xacro:ur_arm_transmission prefix="${tf_prefix}" hw_interface="${transmission_hw_interface}" EE_robotiq="${EE_robotiq}"/>-->
     <!-- Placeholder for ros2_control transmission which don't yet exist -->
     <!-- links -  main serial chain -->
@@ -377,4 +379,303 @@
       <child link="${tf_prefix}tool0"/>
     </joint>
+    <!-- === ROBOTIQ 2f-85 GRIPPER === -->
+    <xacro:if value="${EE_robotiq}">
+      <!-- NOTE: JOINT LIMITS have been slightly augmentated from 0.0 to +-0.05 to avoid errors in MoveIt!2 execution. -->
+      <!-- Robotiq: coupler -->
+      <link name="robotiq_coupler">
+        <visual>
+          <geometry>
+            <mesh filename="file://$(find ur_description)/meshes/robotiq2f85/robotiq_85_coupler.stl" />
+          </geometry>
+        </visual>
+        <collision>
+          <geometry>
+            <mesh filename="file://$(find ur_description)/meshes/robotiq2f85/robotiq_85_coupler.stl" />
+          </geometry>
+        </collision>
+        <inertial>
+          <origin xyz="2.073e-05   1.45286e-03  -1.1049e-03" rpy="0 0 0" />
+          <mass value="0.168" />
+          <inertia ixx="6.69695624e-05" ixy="5.21511788e-09" ixz="-2.74383009e-08"
+                  iyy="7.85088161e-05" iyz="5.41105193e-07" izz="1.41819717e-04"/>
+        </inertial>
+      </link>
+      <joint name="robotiq_coupler_joint" type="fixed">
+        <origin xyz="0 0 0.004" rpy="0 0 ${-pi/2.0}" />
+        <parent link="tool0"/>
+        <child link="robotiq_coupler"/>
+      </joint>
+      <gazebo reference="robotiq_coupler">
+        <mu1>0.9</mu1>
+        <mu2>0.9</mu2>
+        <material>Gazebo/FlatBlack</material>
+      </gazebo>
+      <!-- Robotiq: base_link -->
+      <link name="${tf_prefix}robotiq_85_base_link">
+        <visual>
+          <geometry>
+            <mesh filename="file://$(find ur_description)/meshes/robotiq2f85/visual/robotiq_85_base_link.dae"/>
+          </geometry>
+        </visual>
+        <collision>
+          <geometry>
+            <mesh filename="file://$(find ur_description)/meshes/robotiq2f85/collision/robotiq_85_base_link.stl"/>
+          </geometry>
+        </collision>
+        <inertial>
+          <mass value="0.636951" />
+          <origin xyz="0.0 0.0 0.0" />
+          <inertia ixx = "0.000380" ixy = "0.000000" ixz = "0.000000"
+              iyx = "0.000000" iyy = "0.001110" iyz = "0.000000"
+              izx = "0.000000" izy = "0.000000" izz = "0.001171" />
+        </inertial>
+      </link>
+      <joint name="${tf_prefix}robotiq_85_base_joint" type="fixed">
+        <origin xyz="0 0 0.004" rpy="0 ${-pi/2} ${pi}"/>
+        <parent link="robotiq_coupler"/>
+        <child link="${tf_prefix}robotiq_85_base_link"/>
+      </joint>
+      <!-- Robotiq: left_knuckle -->
+      <link name="${tf_prefix}robotiq_85_left_knuckle_link">
+        <visual>
+          <geometry>
+            <mesh filename="file://$(find ur_description)/meshes/robotiq2f85/visual/robotiq_85_knuckle_link.dae"/>
+          </geometry>
+        </visual>
+        <collision>
+          <geometry>
+            <mesh filename="file://$(find ur_description)/meshes/robotiq2f85/collision/robotiq_85_knuckle_link.stl"/>
+          </geometry>
+        </collision>
+        <inertial>
+          <mass value="0.018491" />
+          <origin xyz="0.0 0.0 0.0" />
+          <inertia ixx = "0.000009" ixy = "-0.000001" ixz = "0.000000"
+              iyx = "-0.000001" iyy = "0.000001" iyz = "0.000000"
+              izx = "0.000000" izy = "0.000000" izz = "0.000010" />
+        </inertial>
+      </link>
+      <joint name="${tf_prefix}robotiq_85_left_knuckle_joint" type="revolute">
+	      <parent link="${tf_prefix}robotiq_85_base_link"/>
+	      <child link="${tf_prefix}robotiq_85_left_knuckle_link"/>
+	      <axis xyz="0 0 1"/>
+	      <origin rpy="${pi} 0.0 0.0" xyz="0.05490451627 0.03060114443 0.0"/>
+	      <limit lower="-0.05" upper="0.80285" velocity="0.5" effort="1000"/>
+        <dynamics damping="1.0" friction="1.0"/>
+	    </joint>
+      <!-- Robotiq: right_knuckle -->
+      <link name="${tf_prefix}robotiq_85_right_knuckle_link">
+        <visual>
+          <geometry>
+            <mesh filename="file://$(find ur_description)/meshes/robotiq2f85/visual/robotiq_85_knuckle_link.dae"/>
+          </geometry>
+        </visual>
+        <collision>
+          <geometry>
+            <mesh filename="file://$(find ur_description)/meshes/robotiq2f85/collision/robotiq_85_knuckle_link.stl"/>
+          </geometry>
+        </collision>
+        <inertial>
+          <mass value="0.018491" />
+          <origin xyz="0.0 0.0 0.0" />
+          <inertia ixx = "0.000009" ixy = "-0.000001" ixz = "0.000000"
+              iyx = "-0.000001" iyy = "0.000001" iyz = "0.000000"
+              izx = "0.000000" izy = "0.000000" izz = "0.000010" />
+        </inertial>
+      </link>
+      <joint name="${tf_prefix}robotiq_85_right_knuckle_joint" type="continuous">
+        <parent link="${tf_prefix}robotiq_85_base_link"/>
+        <child link="${tf_prefix}robotiq_85_right_knuckle_link"/>
+        <axis xyz="0 0 1"/>
+        <origin rpy="0.0 0.0 0.0" xyz="0.05490451627 -0.03060114443 0.0"/>
+        <limit lower="-0.05" upper="0.80285" velocity="0.5" effort="1000"/>
+        <dynamics damping="1.0" friction="1.0"/>
+      </joint>
+      <!-- Robotiq: left_finger -->
+      <link name="${tf_prefix}robotiq_85_left_finger_link">
+        <visual>
+          <geometry>
+            <mesh filename="file://$(find ur_description)/meshes/robotiq2f85/visual/robotiq_85_finger_link.dae"/>
+          </geometry>
+        </visual>
+        <collision>
+          <geometry>
+            <mesh filename="file://$(find ur_description)/meshes/robotiq2f85/collision/robotiq_85_finger_link.stl"/>
+          </geometry>
+        </collision>
+        <inertial>
+          <mass value="0.027309" />
+          <origin xyz="0.0 0.0 0.0" />
+          <inertia ixx = "0.000003" ixy = "-0.000002" ixz = "0.000000"
+              iyx = "-0.000002" iyy = "0.000021" iyz = "0.000000"
+              izx = "0.000000" izy = "0.000000" izz = "0.000020" />
+        </inertial>
+      </link>
+      <joint name="${tf_prefix}robotiq_85_left_finger_joint" type="fixed">
+        <parent link="${tf_prefix}robotiq_85_left_knuckle_link"/>
+        <child link="${tf_prefix}robotiq_85_left_finger_link"/>
+        <origin xyz="-0.00408552455 -0.03148604435 0.0" rpy="0 0 0" />
+        <dynamics damping="1.0" friction="1.0"/>
+      </joint>
+      <!-- Robotiq: right_finger -->
+      <link name="${tf_prefix}robotiq_85_right_finger_link">
+        <visual>
+          <geometry>
+            <mesh filename="file://$(find ur_description)/meshes/robotiq2f85/visual/robotiq_85_finger_link.dae"/>
+          </geometry>
+        </visual>
+        <collision>
+          <geometry>
+            <mesh filename="file://$(find ur_description)/meshes/robotiq2f85/collision/robotiq_85_finger_link.stl"/>
+          </geometry>
+        </collision>
+        <inertial>
+          <mass value="0.027309" />
+          <origin xyz="0.0 0.0 0.0" />
+          <inertia ixx = "0.000003" ixy = "-0.000002" ixz = "0.000000"
+              iyx = "-0.000002" iyy = "0.000021" iyz = "0.000000"
+              izx = "0.000000" izy = "0.000000" izz = "0.000020" />
+        </inertial>
+      </link>
+      <joint name="${tf_prefix}robotiq_85_right_finger_joint" type="fixed">
+        <parent link="${tf_prefix}robotiq_85_right_knuckle_link"/>
+        <child link="${tf_prefix}robotiq_85_right_finger_link"/>
+        <origin xyz="-0.00408552455 -0.03148604435 0.0" rpy="0 0 0" />
+        <dynamics damping="1.0" friction="1.0"/>
+      </joint>
+      <!-- Robotiq: left_inner_knuckle -->
+      <link name="${tf_prefix}robotiq_85_left_inner_knuckle_link">
+        <visual>
+          <geometry>
+            <mesh filename="file://$(find ur_description)/meshes/robotiq2f85/visual/robotiq_85_inner_knuckle_link.dae"/>
+          </geometry>
+        </visual>
+        <collision>
+          <geometry>
+            <mesh filename="file://$(find ur_description)/meshes/robotiq2f85/collision/robotiq_85_inner_knuckle_link.stl"/>
+          </geometry>
+        </collision>
+        <inertial>
+          <mass value="0.029951" />
+          <origin xyz="0.0 0.0 0.0" />
+          <inertia ixx = "0.000039" ixy = "0.000000" ixz = "0.000000"
+              iyx = "0.000000" iyy = "0.000005" iyz = "0.000000"
+              izx = "0.000000" izy = "0.000000" izz = "0.000035" />
+        </inertial>
+      </link>
+      <joint name="${tf_prefix}robotiq_85_left_inner_knuckle_joint" type="continuous">
+        <parent link="${tf_prefix}robotiq_85_base_link"/>
+        <child link="${tf_prefix}robotiq_85_left_inner_knuckle_link"/>
+        <axis xyz="0 0 1"/>
+        <origin xyz="0.06142 0.0127 0" rpy="${pi} 0.0 0.0" />
+        <limit lower="-0.05" upper="0.80285" velocity="0.5" effort="1000"/>
+        <dynamics damping="1.0" friction="1.0"/>
+      </joint>
+      <!-- Robotiq: right_inner_knuckle -->
+      <link name="${tf_prefix}robotiq_85_right_inner_knuckle_link">
+        <visual>
+          <geometry>
+            <mesh filename="file://$(find ur_description)/meshes/robotiq2f85/visual/robotiq_85_inner_knuckle_link.dae"/>
+          </geometry>
+        </visual>
+        <collision>
+          <geometry>
+            <mesh filename="file://$(find ur_description)/meshes/robotiq2f85/collision/robotiq_85_inner_knuckle_link.stl"/>
+          </geometry>
+        </collision>
+        <inertial>
+          <mass value="0.029951" />
+          <origin xyz="0.0 0.0 0.0" />
+          <inertia ixx = "0.000039" ixy = "0.000000" ixz = "0.000000"
+              iyx = "0.000000" iyy = "0.000005" iyz = "0.000000"
+              izx = "0.000000" izy = "0.000000" izz = "0.000035" />
+        </inertial>
+      </link>
+      <joint name="${tf_prefix}robotiq_85_right_inner_knuckle_joint" type="continuous">
+        <parent link="${tf_prefix}robotiq_85_base_link"/>
+        <child link="${tf_prefix}robotiq_85_right_inner_knuckle_link"/>
+        <axis xyz="0 0 1"/>
+        <origin xyz="0.06142 -0.0127 0" rpy="0 0 0"/>
+        <limit lower="-0.05" upper="0.80285" velocity="0.5" effort="1000"/>
+        <dynamics damping="1.0" friction="1.0"/>
+      </joint>
+      <!-- Robotiq: left_finger_tip -->
+      <link name="${tf_prefix}robotiq_85_left_finger_tip_link">
+        <visual>
+          <geometry>
+            <mesh filename="file://$(find ur_description)/meshes/robotiq2f85/visual/robotiq_85_finger_tip_link.dae"/>
+          </geometry>
+        </visual>
+        <collision>
+          <geometry>
+            <mesh filename="file://$(find ur_description)/meshes/robotiq2f85/collision/robotiq_85_finger_tip_link.stl"/>
+          </geometry>
+        </collision>
+        <inertial>
+          <mass value="0.019555" />
+          <origin xyz="0.0 0.0 0.0" />
+          <inertia ixx = "0.000002" ixy = "0.000000" ixz = "0.000000"
+              iyx = "0.000000" iyy = "0.000005" iyz = "0.000000"
+              izx = "0.000000" izy = "0.000000" izz = "0.000006" />
+        </inertial>
+      </link>
+      <joint name="${tf_prefix}robotiq_85_left_finger_tip_joint" type="continuous">
+        <parent link="${tf_prefix}robotiq_85_left_inner_knuckle_link"/>
+        <child link="${tf_prefix}robotiq_85_left_finger_tip_link"/>
+        <axis xyz="0 0 1"/>
+        <origin xyz="0.04303959807 -0.03759940821 0.0" rpy="0.0 0.0 0.0"/>
+        <limit lower="-0.80285" upper="0.05" velocity="0.5" effort="1000"/>
+        <dynamics damping="1.0" friction="1.0"/>
+      </joint>
+      <!-- Robotiq: right_finger_tip -->
+      <link name="${tf_prefix}robotiq_85_right_finger_tip_link">
+        <visual>
+          <geometry>
+            <mesh filename="file://$(find ur_description)/meshes/robotiq2f85/visual/robotiq_85_finger_tip_link.dae"/>
+          </geometry>
+        </visual>
+        <collision>
+          <geometry>
+            <mesh filename="file://$(find ur_description)/meshes/robotiq2f85/collision/robotiq_85_finger_tip_link.stl"/>
+          </geometry>
+        </collision>
+        <inertial>
+          <mass value="0.019555" />
+          <origin xyz="0.0 0.0 0.0" />
+          <inertia ixx = "0.000002" ixy = "0.000000" ixz = "0.000000"
+              iyx = "0.000000" iyy = "0.000005" iyz = "0.000000"
+              izx = "0.000000" izy = "0.000000" izz = "0.000006" />
+        </inertial>
+      </link>
+      <joint name="${tf_prefix}robotiq_85_right_finger_tip_joint" type="continuous">
+        <parent link="${tf_prefix}robotiq_85_right_inner_knuckle_link"/>
+        <child link="${tf_prefix}robotiq_85_right_finger_tip_link"/>
+        <axis xyz="0 0 1"/>
+        <origin rpy="0.0 0.0 0.0" xyz="0.04303959807 -0.03759940821  0.0"/>
+        <limit lower="-0.80285" upper="0.05" velocity="0.5" effort="1000"/>
+        <dynamics damping="1.0" friction="1.0"/>
+      </joint>
+      <!-- SMALL CUBE FOR GRIPPER PLUGIN -->
+      <link name="EE_robotiq_2f85">
+        <inertial>
+          <origin xyz="0 0 0" rpy="0 0 0" />
+          <mass value="0.00001" />
+          <inertia ixx="0.001" ixy="0.0" ixz="0.0" iyy="0.001" iyz="0.0" izz="0.001"/>
+        </inertial>
+        <visual>
+          <geometry>
+            <box size= "0.001 0.001 0.001" />
+          </geometry>
+        </visual>
+      </link>
+      <joint name="EE_robotiq_2f85_joint" type="prismatic" >
+        <parent link="${tf_prefix}robotiq_85_base_link" />
+        <child link="EE_robotiq_2f85" />
+        <limit effort="10000" lower="0.0" upper="0.0" velocity="0.0"/>
+        <axis xyz="1 0 0" />
+        <origin xyz="0.128 0.0 0.0" rpy="0 0 0"/>
+      </joint>
+    </xacro:if>
+    <!-- === ROBOTIQ 2f-85 GRIPPER === -->
   </xacro:macro>
 </robot>
