Commit message: able to launch ur5 with gripper to gazebo
Signed-off-by: Roshan Kumar <rkroshan.1999@gmail.com>

File: urdf/ur.urdf.xacro (robot description, xacro)
@@ -100,4 +100,5 @@
       <plugin filename="libgazebo_ros2_control.so" name="gazebo_ros2_control">
         <robot_sim_type>gazebo_ros2_control/GazeboSystem</robot_sim_type>
+        <parameters>$(arg simulation_controllers)</parameters>
         <parameters>$(find ur_description)/config/urrobotiq_controller.yaml</parameters>
       </plugin>

File: urdf/ur_macro.xacro (robot description, xacro)
@@ -657,5 +657,5 @@
       </joint>
       <!-- SMALL CUBE FOR GRIPPER PLUGIN -->
-      <link name="EE_robotiq_2f85">
+      <!-- <link name="EE_robotiq_2f85">
         <inertial>
           <origin xyz="0 0 0" rpy="0 0 0" />
@@ -675,5 +675,5 @@
         <axis xyz="1 0 0" />
         <origin xyz="0.128 0.0 0.0" rpy="0 0 0"/>
-      </joint>
+      </joint> -->
     </xacro:if>
     <!-- === ROBOTIQ 2f-85 GRIPPER === -->
